File: HexDisplayPCB.kicad_pcb (KiCad board)
At the start: 2 copper layers, 259.8 x 300 mm, 79 parts, among them J1 Conn_01x20, J2 Conn_01x20, J3 Conn_01x16, J30 Barrel_Jack_Switch, J4 Conn_01x16, J5 Conn_01x16, J6 Conn_01x16, J7 Conn_01x16, J8 Conn_01x16, U1 SN74HCT245DWR

Commit message: Final first draft with gerber
Parts:
- removed 3V3_IN_1-4, 3V3_IN_5-8, 5V_OUT_1-4, 5V_OUT_4-8: Conn_01x04, Connector_PinSocket_2.54mm:PinSocket_1x04_P2.54mm_Vertical
- removed DATA_1_DISCONNECT_2, DATA_2_DISCONNECT_2, DATA_3_DISCONNECT_2, DATA_4_DISCONNECT_2, DATA_5_DISCONNECT_2, DATA_6_DISCONNECT_2, SCL-DATA_8, SDA-DATA_7: SolderJumper_2_Open, Jumper:SolderJumper-2_P1.3mm_Open_TrianglePad1.0x1.5mm
- added STEPPER_1-4: Conn_01x08, Connector_PinHeader_2.54mm:PinHeader_1x08_P2.54mm_Vertical, B.Cu at (452.1, 246.4)
- added STEPPER_4-8: Conn_01x08, Connector_PinHeader_2.54mm:PinHeader_1x08_P2.54mm_Vertical, B.Cu at (467.4, 246.4)
- moved LED_DATA_IN-DATA_1 178.0 mm to (404.4, 238.3), turned to 0 degrees
- moved LED_DATA_IN-DATA_2 178.0 mm to (404.4, 241.8), turned to 0 degrees
- moved LED_DATA_IN-DATA_3 178.0 mm to (404.4, 245.4), turned to 0 degrees
- moved LED_DATA_IN-DATA_4 178.0 mm to (404.4, 248.9), turned to 0 degrees
- moved LED_DATA_IN-DATA_5 178.0 mm to (404.4, 252.5), turned to 0 degrees
- moved LED_DATA_IN-DATA_6 178.0 mm to (404.4, 256.0), turned to 0 degrees
- moved U1 15.2 mm to (459.6, 250.2)
- moved LED_DATA_OUT1 3.81 mm to (453.4, 279.4)
- moved A14 0.15 mm to (399.2, 128.0)
- turned PICO_DATAIN_5-STEPPER1 to 0 degrees
- turned PICO_DATAIN_6-STEPPER1 to 0 degrees
- turned STEPPER-DATA_5 to 180 degrees
- turned STEPPER-DATA_6 to 180 degrees
Connections:
- DATA_1_DISCONNECT_1 pad 2: Net-(DATA_1_DISCONNECT_1-B) -> /BUS_1
- DATA_2_DISCONNECT_1 pad 2: Net-(DATA_2_DISCONNECT_1-B) -> /BUS_2
- DATA_3_DISCONNECT_1 pad 2: Net-(DATA_3_DISCONNECT_1-B) -> /BUS_3
- DATA_4_DISCONNECT_1 pad 2: Net-(DATA_4_DISCONNECT_1-B) -> /BUS_4
- DATA_5_DISCONNECT_1 pad 2: Net-(DATA_5_DISCONNECT_1-B) -> /BUS_5
- DATA_6_DISCONNECT_1 pad 2: Net-(DATA_6_DISCONNECT_1-B) -> /BUS_6
- J3 pad 1: Net-(DATA_1_DISCONNECT_1-B) -> /BUS_1
- J3 pad 11: Net-(DATA_6_DISCONNECT_2-B) -> /BUS_6
- J3 pad 12: Net-(DATA_5_DISCONNECT_2-B) -> /BUS_5
- J3 pad 13: Net-(DATA_4_DISCONNECT_2-B) -> /BUS_4
- J3 pad 14: Net-(DATA_3_DISCONNECT_2-B) -> /BUS_3
- J3 pad 15: Net-(DATA_2_DISCONNECT_2-B) -> /BUS_2
- J3 pad 16: Net-(DATA_1_DISCONNECT_2-B) -> /BUS_1
- J3 pad 2: Net-(DATA_2_DISCONNECT_1-B) -> /BUS_2
- J3 pad 3: Net-(DATA_3_DISCONNECT_1-B) -> /BUS_3
- J3 pad 4: Net-(DATA_4_DISCONNECT_1-B) -> /BUS_4
- J3 pad 5: Net-(DATA_5_DISCONNECT_1-B) -> /BUS_5
- J3 pad 6: Net-(DATA_6_DISCONNECT_1-B) -> /BUS_6
- J4 pad 1: Net-(DATA_1_DISCONNECT_1-B) -> /BUS_1
- J4 pad 11: Net-(DATA_6_DISCONNECT_2-B) -> /BUS_6
- J4 pad 12: Net-(DATA_5_DISCONNECT_2-B) -> /BUS_5
- J4 pad 13: Net-(DATA_4_DISCONNECT_2-B) -> /BUS_4
- J4 pad 14: Net-(DATA_3_DISCONNECT_2-B) -> /BUS_3
- J4 pad 15: Net-(DATA_2_DISCONNECT_2-B) -> /BUS_2
- J4 pad 16: Net-(DATA_1_DISCONNECT_2-B) -> /BUS_1
- J4 pad 2: Net-(DATA_2_DISCONNECT_1-B) -> /BUS_2
- J4 pad 3: Net-(DATA_3_DISCONNECT_1-B) -> /BUS_3
- J4 pad 4: Net-(DATA_4_DISCONNECT_1-B) -> /BUS_4
- J4 pad 5: Net-(DATA_5_DISCONNECT_1-B) -> /BUS_5
- J4 pad 6: Net-(DATA_6_DISCONNECT_1-B) -> /BUS_6
- J5 pad 1: Net-(DATA_1_DISCONNECT_1-B) -> /BUS_1
- J5 pad 11: Net-(DATA_6_DISCONNECT_2-B) -> /BUS_6
- J5 pad 12: Net-(DATA_5_DISCONNECT_2-B) -> /BUS_5
- J5 pad 13: Net-(DATA_4_DISCONNECT_2-B) -> /BUS_4
- J5 pad 14: Net-(DATA_3_DISCONNECT_2-B) -> /BUS_3
- J5 pad 15: Net-(DATA_2_DISCONNECT_2-B) -> /BUS_2
- J5 pad 16: Net-(DATA_1_DISCONNECT_2-B) -> /BUS_1
- J5 pad 2: Net-(DATA_2_DISCONNECT_1-B) -> /BUS_2
- J5 pad 3: Net-(DATA_3_DISCONNECT_1-B) -> /BUS_3
- J5 pad 4: Net-(DATA_4_DISCONNECT_1-B) -> /BUS_4
- J5 pad 5: Net-(DATA_5_DISCONNECT_1-B) -> /BUS_5
- J5 pad 6: Net-(DATA_6_DISCONNECT_1-B) -> /BUS_6
- J6 pad 1: Net-(DATA_1_DISCONNECT_1-B) -> /BUS_1
- J6 pad 11: Net-(DATA_6_DISCONNECT_2-B) -> /BUS_6
- J6 pad 12: Net-(DATA_5_DISCONNECT_2-B) -> /BUS_5
- J6 pad 13: Net-(DATA_4_DISCONNECT_2-B) -> /BUS_4
- J6 pad 14: Net-(DATA_3_DISCONNECT_2-B) -> /BUS_3
- J6 pad 15: Net-(DATA_2_DISCONNECT_2-B) -> /BUS_2
- J6 pad 16: Net-(DATA_1_DISCONNECT_2-B) -> /BUS_1
- J6 pad 2: Net-(DATA_2_DISCONNECT_1-B) -> /BUS_2
- J6 pad 3: Net-(DATA_3_DISCONNECT_1-B) -> /BUS_3
- J6 pad 4: Net-(DATA_4_DISCONNECT_1-B) -> /BUS_4
- J6 pad 5: Net-(DATA_5_DISCONNECT_1-B) -> /BUS_5
- J6 pad 6: Net-(DATA_6_DISCONNECT_1-B) -> /BUS_6
- J7 pad 1: Net-(DATA_1_DISCONNECT_1-B) -> /BUS_1
- J7 pad 11: Net-(DATA_6_DISCONNECT_2-B) -> /BUS_6
- J7 pad 12: Net-(DATA_5_DISCONNECT_2-B) -> /BUS_5
- J7 pad 13: Net-(DATA_4_DISCONNECT_2-B) -> /BUS_4
- J7 pad 14: Net-(DATA_3_DISCONNECT_2-B) -> /BUS_3
- J7 pad 15: Net-(DATA_2_DISCONNECT_2-B) -> /BUS_2
- J7 pad 16: Net-(DATA_1_DISCONNECT_2-B) -> /BUS_1
- J7 pad 2: Net-(DATA_2_DISCONNECT_1-B) -> /BUS_2
- J7 pad 3: Net-(DATA_3_DISCONNECT_1-B) -> /BUS_3
- J7 pad 4: Net-(DATA_4_DISCONNECT_1-B) -> /BUS_4
- J7 pad 5: Net-(DATA_5_DISCONNECT_1-B) -> /BUS_5
- J7 pad 6: Net-(DATA_6_DISCONNECT_1-B) -> /BUS_6
- J8 pad 1: Net-(DATA_1_DISCONNECT_1-B) -> /BUS_1
- J8 pad 11: Net-(DATA_6_DISCONNECT_2-B) -> /BUS_6
- J8 pad 12: Net-(DATA_5_DISCONNECT_2-B) -> /BUS_5
- J8 pad 13: Net-(DATA_4_DISCONNECT_2-B) -> /BUS_4
- J8 pad 14: Net-(DATA_3_DISCONNECT_2-B) -> /BUS_3
- J8 pad 15: Net-(DATA_2_DISCONNECT_2-B) -> /BUS_2
- J8 pad 16: Net-(DATA_1_DISCONNECT_2-B) -> /BUS_1
- J8 pad 2: Net-(DATA_2_DISCONNECT_1-B) -> /BUS_2
- J8 pad 3: Net-(DATA_3_DISCONNECT_1-B) -> /BUS_3
- J8 pad 4: Net-(DATA_4_DISCONNECT_1-B) -> /BUS_4
- J8 pad 5: Net-(DATA_5_DISCONNECT_1-B) -> /BUS_5
- J8 pad 6: Net-(DATA_6_DISCONNECT_1-B) -> /BUS_6
- U2 pad 12: /KEYPAD_5 -> unconnected-(U2-R3-Pad12)
- U2 pad 13: GND -> /KEYPAD_5
- U2 pad 14: unconnected-(U2-C9-Pad14) -> GND
- U2 pad 20: /KEYPAD_1 -> unconnected-(U2-C4-Pad20)
- U2 pad 21: /KEYPAD_2 -> /KEYPAD_1
- U2 pad 22: /KEYPAD_3 -> /KEYPAD_2
- U2 pad 23: /KEYPAD_4 -> /KEYPAD_3
- U2 pad 24: /KEYPAD_6 -> /KEYPAD_4
- U2 pad 25: /KEYPAD_7 -> /KEYPAD_6
- U2 pad 26: (no net) -> /KEYPAD_7
Routing:
- net GND: track 0.00 -> 2150.3 mm, vias 0 -> 43
- net +5V: track 0.00 -> 1604.5 mm, vias 0 -> 29
- net /BUS_1: track 0.00 -> 885.5 mm, vias 0 -> 3
- net /BUS_2: track 0.00 -> 849.9 mm, vias 0 -> 5
- net /BUS_3: track 0.00 -> 828.4 mm, vias 0 -> 5
- net /BUS_4: track 0.00 -> 803.3 mm, vias 0 -> 5
- net /BUS_5: track 0.00 -> 779.3 mm, vias 0 -> 5
- net /BUS_6: track 0.00 -> 757.5 mm, vias 0 -> 5
- net +3V3: track 0.00 -> 489.5 mm, vias 0 -> 5
- net /SCL: track 0.00 -> 482.6 mm, vias 0 -> 3
- net /SDA: track 0.00 -> 465.9 mm, vias 0 -> 3
- net /KEYPAD_INT: track 0.00 -> 338.1 mm, vias 0 -> 1
- net /SWCLK: track 0.00 -> 331.7 mm
- net /SWDIO: track 0.00 -> 324.9 mm
- net /UART0 RX: track 0.00 -> 273.6 mm, vias 0 -> 3
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Other:
- outline, holes or cut-outs redrawn

Commit message: Final image adjustments
Parts:
- added G***: LOGO, Feesh:Feesh, F.Cu at (440.8, 294.9)
- moved AmbientLightSensor1 6.11 mm to (363.5, 90.8)
Connections:
- AmbientLightSensor1 pad 2: GND -> unconnected-(AmbientLightSensor1-Pin_2-Pad2)
- AmbientLightSensor1 pad 3: /SCL -> GND
- AmbientLightSensor1 pad 4: /SDA -> /SCL
- AmbientLightSensor1 pad 5: unconnected-(AmbientLightSensor1-Pin_5-Pad5) -> /SDA
Routing:
- net +3V3: track 489.5 -> 502.4 mm
- net +5V: track 1604.5 -> 1617.4 mm, vias 29 -> 28
- net GND: track 2150.3 -> 2139.6 mm, vias 43 -> 46
- net /SDA: track 465.9 -> 464.3 mm
- net /SCL: track 482.6 -> 481.7 mm
Other:
- board text added: "HEX DISPLAY PCB V1"
